File: kicad/arduino-lab.kicad_pcb (KiCad board)
At the start: 2 copper layers, 68.6 x 100 mm, 22 parts, among them J1 joystick, J2 Conn_01x03, J3 Conn_01x03, J4 Conn_01x04, SW1 SW_Push, SW2 SW_Push, SW3 SW_Push, U1 TXB0104D

Commit message: Added kicad files
Connections:
- XA1 pad D10: SERVO2 -> Net-(XA1-PadD10)
- XA1 pad D11: Net-(XA1-PadD11) -> SERVO2
Routing:
- net SERVO2: track 63.7 -> 64.8 mm
- net VIN: track 129.4 -> 128.5 mm
- net 5V: track 156.3 -> 157.1 mm
